Commit message: updated

File: urdf/haul_truck.urdf (robot description, URDF)
Before this commit: robot haul truck, 6 links, 5 joints
Links:
- link back_left_wheel: geometry visual mesh filename=package://truck/meshes/parts_Wheel.dae
- link back_right_wheel: geometry visual mesh filename=package://truck/meshes/parts_Wheel.dae
- link left_wheel: geometry visual mesh filename=package://truck/meshes/parts_Wheel.dae
- link right_wheel: geometry visual mesh filename=package://truck/meshes/parts_Wheel.dae

Commit message: Updating models

File: urdf/haul_truck.urdf (robot description, URDF)
Before this commit: robot haul truck, 6 links, 5 joints
Links:
- link base_link: geometry collision mesh filename=package://truck/meshes/parts_Body.dae; visual mesh filename=package://truck/meshes/parts_Body.dae
- link tray: geometry collision mesh filename=package://truck/meshes/parts_Tray23.dae; visual mesh filename=package://truck/meshes/parts_Tray23.dae

Commit message: updated haul truck joint origins

File: urdf/haul_truck.urdf (robot description, URDF)
Before this commit: robot haul truck, 6 links, 5 joints
Joints:
- joint back_left_wheel_joint: axis 0 0 1 -> 1 0 0; limit lower=0.0 upper=0.0 effort=0.0 velocity=0.0 -> (none); origin xyz=4.9 4.0 0.0 rpy=0.0 -0.0 3.141592653589793 -> xyz=2.0 6.0 0.0 rpy=0.0 -0.0 3.141592653589793; type revolute -> continuous
- joint back_right_wheel_joint: axis 0 0 1 -> 1 0 0; limit lower=0.0 upper=0.0 effort=0.0 velocity=0.0 -> (none); origin xyz=0.0 4.0 0.0 rpy=0.0 -0.0 0.0 -> xyz=-2.0 6.0 0.0 rpy=0.0 -0.0 0.0; type revolute -> continuous
- joint body_to_tray_joint: limit lower=0.0 upper=0.0 effort=0.0 velocity=0.0 -> (none); type revolute -> fixed
- joint left_wheel_joint: axis 0 0 1 -> 1 0 0; limit lower=0.0 upper=0.0 effort=0.0 velocity=0.0 -> (none); origin xyz=4.9 0.0 0.0 rpy=0.0 -0.0 3.141592653589793 -> xyz=2.0 1.5 0.0 rpy=0.0 -0.0 3.141592653589793; type revolute -> continuous
- joint right_wheel_joint: axis 0 0 1 -> 1 0 0; limit lower=0.0 upper=0.0 effort=0.0 velocity=0.0 -> (none); origin xyz=0.0 0.0 0.0 rpy=0.0 -0.0 0.0 -> xyz=-2.0 1.5 0.0 rpy=0.0 -0.0 0.0; type revolute -> continuous
